Commit message: urdf file with both arms, need exact pose for both arms

File: tufts_urdf_setup/UR5/00-ur5frame.urdf (robot description, URDF)
Before this commit: robot ur5, 2 links, 2 joints
Joints:
- removed joint world_joint
- added joint world_joint_1: type fixed, parent ur5_frame, child base_link, origin xyz=0.607 0.635 1.27 rpy=${0*pi/180} ${135*pi/180}  ${0*pi/180}
- added joint world_joint_2: type fixed, parent ur5_frame, child 2_base_link

Commit message: updated urdf file for ur5 setup

File: tufts_urdf_setup/UR5/00-ur5frame.urdf (robot description, URDF)
Before this commit: robot ur5, 2 links, 3 joints
Joints:
- joint world_joint_2: origin (none) -> xyz=0.28 0.69 1.27 rpy=${0*pi/180} ${225*pi/180}  ${0*pi/180}

Commit message: updated arm position on frame

File: tufts_urdf_setup/UR5/00-ur5frame.urdf (robot description, URDF)
Before this commit: robot ur5, 2 links, 3 joints
Joints:
- joint world_joint_1: child base_link -> left_base_link; origin xyz=0.607 0.635 1.27 rpy=${0*pi/180} ${135*pi/180}  ${0*pi/180} -> xyz=0.645 0.635 1.275 rpy=${0*pi/180} ${135*pi/180}  ${0*pi/180}
- joint world_joint_2: child 2_base_link -> right_base_link; origin xyz=0.28 0.69 1.27 rpy=${0*pi/180} ${225*pi/180}  ${0*pi/180} -> xyz=0.265 0.635 1.275 rpy=${0*pi/180} ${225*pi/180}  ${0*pi/180}
